Commit message: Create 4 DOF robot URDF file Create tf broadcaster for robot Direct transforms to joints

File: src/rrm_cv3_pal/urdf/arm.urdf (robot description, URDF)
Before this commit: robot arm, 6 links, 5 joints
Links:
- removed link joint_1
- removed link joint_2
- removed link link1
- removed link link2
- added link link_ball_1; visual sphere radius=0.03
- added link link_ball_2; visual sphere radius=0.03
- added link link_ball_3; visual sphere radius=0.03
- added link link_ball_4; visual sphere radius=0.03
- added link link_vis_1; visual cylinder length=0.203 radius=0.01
- added link link_vis_2; visual cylinder length=0.203 radius=0.01
- added link link_vis_3; visual cylinder length=0.203 radius=0.01
- added link link_vis_3B; visual cylinder length=0.203 radius=0.01
- added link link_vis_4; visual cylinder length=0.178 radius=0.01
Joints:
- removed joint joint_2_to_tool0
- removed joint link1_to_joint_1
- removed joint link2_to_joint_2
- added joint joint_3: type prismatic, parent link_ball_2, child link_ball_3, origin xyz=0 0 0.203 rpy=0 0 0, axis 0 0 1, limit lower=0 upper=0.15 effort=1000.0 velocity=0.5
- added joint joint_4: type revolute, parent link_ball_3, child link_ball_4, origin xyz=0 0 0.203 rpy=0 0 0, axis 0 1 0, limit lower=-0.96 upper=2.182 effort=1000.0 velocity=0.5
- added joint joint_to_tool0: type fixed, parent link_ball_4, child tool0, origin xyz=0 0 0.178 rpy=0 0 0
- added joint joint_vis_1: type fixed, parent link_ball_1, child link_vis_1, origin xyz=0 0 0.1015 rpy=0 0 0
- added joint joint_vis_2: type fixed, parent link_ball_2, child link_vis_2, origin xyz=0 0 0.089 rpy=0 0 0
- added joint joint_vis_3: type fixed, parent link_ball_3, child link_vis_3, origin xyz=0 0 0.089 rpy=0 0 0
- added joint joint_vis_3B: type fixed, parent link_ball_3, child link_vis_3B, origin xyz=0 0 -0.1 rpy=0 0 0
- added joint joint_vis_4: type fixed, parent link_ball_4, child link_vis_4, origin xyz=0 0 0.089 rpy=0 0 0
- joint joint_1: child joint_1 -> link_ball_1
- joint joint_2: child joint_2 -> link_ball_2; parent joint_1 -> link_ball_1
