Commit message: add laser to robot, speed up robot_state_publisher

File: src/abb_camera_simulation/urdf/abb_irb4600_60_205_macro.xacro (robot description, xacro)
@@ -2,5 +2,5 @@
 <robot xmlns:xacro="http://ros.org/wiki/xacro">
     <xacro:macro name="abb_irb4600_60_205" params="prefix">
-    <!-- link list -->
+        <!-- link list -->
         <link name="world"/>
         <joint name="to_world" type="fixed">
@@ -20,5 +20,5 @@
             </visual>
             <collision>
-            <origin xyz="0 0 0" rpy="0 0 0" />
+                <origin xyz="0 0 0" rpy="0 0 0" />
                 <geometry>
                     <mesh filename="package://abb_camera_simulation/meshes/abb_irb4600_60_205/collision/base_link.stl"/>
@@ -26,37 +26,31 @@
                 <material name="yellow">
                     <color rgba="0 1 1 1"/>
-            </material>
-            </collision>
-            <inertial>
-                  <origin xyz="0 0 0" rpy="0 0 0"/>
-                  <mass value="1"/>
-                  <inertia
-            	  ixx="0.01" ixy="0.01" ixz="0.01"
-            	  iyy="0.01" iyz="0.01"
-            	  izz="0.01"/>
+                </material>
+            </collision>
+            <inertial>
+                <origin xyz="0 0 0" rpy="0 0 0"/>
+                <mass value="1"/>
+                <inertia ixx="0.01" ixy="0.01" ixz="0.01" iyy="0.01" iyz="0.01" izz="0.01"/>
             </inertial>
         </link>
         <link name="${prefix}link_1">
             <visual>
-              <origin xyz="0 0 0" rpy="0 0 0" />
-              <geometry>
-                <mesh filename="package://abb_camera_simulation/meshes/abb_irb4600_60_205/visual/link_1.stl"/>
-              </geometry>
-              <material name="abb_white"/>
-            </visual>
-            <collision>
-             <origin xyz="0 0 0" rpy="0 0 0" />
-            <geometry>
-              <mesh filename="package://abb_camera_simulation/meshes/abb_irb4600_60_205/collision/link_1.stl"/>
-            </geometry>
-            <material name="yellow"/>
-            </collision>
-            <inertial>
-                  <origin xyz="0 0 0" rpy="0 0 0"/>
-                  <mass value="1"/>
-                  <inertia
-            	  ixx="0.01" ixy="0.01" ixz="0.01"
-            	  iyy="0.01" iyz="0.01"
-            	  izz="0.01"/>
+                <origin xyz="0 0 0" rpy="0 0 0" />
+                <geometry>
+                    <mesh filename="package://abb_camera_simulation/meshes/abb_irb4600_60_205/visual/link_1.stl"/>
+                </geometry>
+                <material name="abb_white"/>
+            </visual>
+            <collision>
+                <origin xyz="0 0 0" rpy="0 0 0" />
+                <geometry>
+                    <mesh filename="package://abb_camera_simulation/meshes/abb_irb4600_60_205/collision/link_1.stl"/>
+                </geometry>
+                <material name="yellow"/>
+            </collision>
+            <inertial>
+                <origin xyz="0 0 0" rpy="0 0 0"/>
+                <mass value="1"/>
+                <inertia ixx="0.01" ixy="0.01" ixz="0.01" iyy="0.01" iyz="0.01" izz="0.01"/>
             </inertial>
         </link>
@@ -77,10 +71,7 @@
             </collision>
             <inertial>
-                  <origin xyz="0 0 0" rpy="0 0 0"/>
-                  <mass value="1"/>
-                  <inertia
-            	  ixx="0.01" ixy="0.01" ixz="0.01"
-            	  iyy="0.01" iyz="0.01"
-            	  izz="0.01"/>
+                <origin xyz="0 0 0" rpy="0 0 0"/>
+                <mass value="1"/>
+                <inertia ixx="0.01" ixy="0.01" ixz="0.01" iyy="0.01" iyz="0.01" izz="0.01"/>
             </inertial>
         </link>
@@ -101,10 +92,7 @@
             </collision>
             <inertial>
-                  <origin xyz="0 0 0" rpy="0 0 0"/>
-                  <mass value="1"/>
-                  <inertia
-            	  ixx="0.01" ixy="0.01" ixz="0.01"
-            	  iyy="0.01" iyz="0.01"
-            	  izz="0.01"/>
+                <origin xyz="0 0 0" rpy="0 0 0"/>
+                <mass value="1"/>
+                <inertia ixx="0.01" ixy="0.01" ixz="0.01" iyy="0.01" iyz="0.01" izz="0.01"/>
             </inertial>
         </link>
@@ -125,10 +113,7 @@
             </collision>
             <inertial>
-                  <origin xyz="0 0 0" rpy="0 0 0"/>
-                  <mass value="1"/>
-                  <inertia
-            	  ixx="0.01" ixy="0.01" ixz="0.01"
-            	  iyy="0.01" iyz="0.01"
-            	  izz="0.01"/>
+                <origin xyz="0 0 0" rpy="0 0 0"/>
+                <mass value="1"/>
+                <inertia ixx="0.01" ixy="0.01" ixz="0.01" iyy="0.01" iyz="0.01" izz="0.01"/>
             </inertial>
         </link>
@@ -149,10 +134,7 @@
             </collision>
             <inertial>
-                  <origin xyz="0 0 0" rpy="0 0 0"/>
-                  <mass value="1"/>
-                  <inertia
-            	  ixx="0.01" ixy="0.01" ixz="0.01"
-            	  iyy="0.01" iyz="0.01"
-            	  izz="0.01"/>
+                <origin xyz="0 0 0" rpy="0 0 0"/>
+                <mass value="1"/>
+                <inertia ixx="0.01" ixy="0.01" ixz="0.01" iyy="0.01" iyz="0.01" izz="0.01"/>
             </inertial>
         </link>
@@ -168,17 +150,14 @@
             </visual>
             <collision>
-               <origin xyz="0 0 0" rpy="0 0 0" />
-                  <geometry>
-                     <mesh filename="package://abb_camera_simulation/meshes/abb_irb4600_60_205/collision/link_6.stl"/>
-                  </geometry>
-                  <material name="yellow"/>
-            </collision>
-            <inertial>
-                  <origin xyz="0 0 0" rpy="0 0 0"/>
-                  <mass value="1"/>
-                  <inertia
-            	  ixx="0.01" ixy="0.01" ixz="0.01"
-            	  iyy="0.01" iyz="0.01"
-            	  izz="0.01"/>
+                <origin xyz="0 0 0" rpy="0 0 0" />
+                <geometry>
+                    <mesh filename="package://abb_camera_simulation/meshes/abb_irb4600_60_205/collision/link_6.stl"/>
+                </geometry>
+                <material name="yellow"/>
+            </collision>
+            <inertial>
+                <origin xyz="0 0 0" rpy="0 0 0"/>
+                <mass value="1"/>
+                <inertia ixx="0.01" ixy="0.01" ixz="0.01" iyy="0.01" iyz="0.01" izz="0.01"/>
             </inertial>
         </link>
@@ -204,8 +183,5 @@
                 <origin xyz="0 0 0" rpy="0 0 0"/>
                 <mass value="0.1"/>
-                <inertia
-                        ixx="0.01" ixy="0.01" ixz="0.01"
-                        iyy="0.01" iyz="0.01"
-                        izz="0.01"/>
+                <inertia ixx="0.01" ixy="0.01" ixz="0.01" iyy="0.01" iyz="0.01" izz="0.01"/>
             </inertial>
         </link>
@@ -226,5 +202,5 @@
         </joint>
         <joint name="${prefix}joint_2" type="revolute">
-        <origin xyz="0.174999999999998 -0.0515489073390827 0.341500000000001" rpy="-1.57772181044202E-30 0 0" />
+            <origin xyz="0.174999999999998 -0.0515489073390827 0.341500000000001" rpy="-1.57772181044202E-30 0 0" />
             <parent link="${prefix}link_1"/>
             <child link="${prefix}link_2"/>
@@ -263,23 +239,10 @@
             <parent link="${prefix}link_6"/>
             <child link="${prefix}tool0"/>
-            <origin xyz="0.135 0 0" rpy="0 1.570796 0"/>
+            <origin xyz="0.135 0 0" rpy="0 0 0"/>
         </joint>
         <joint name="to_kinect" type="fixed">
             <parent link="${prefix}tool0"/>
             <child link="kinect_frame"/>
-            Translation
-            -0.0694681
-            -0.284737
-            0.247462
-            Rotation
-            -1.61514
-            -0.043724
-            -2.17802
-            <origin xyz="-0.0695877
- -0.285281
-  0.240969"
-                    rpy=" -1.61039
--0.0438775
-  -2.17805"/>
+            <origin xyz="-0.0695877 -0.285281 0.240969" rpy=" -1.61039 -0.0438775 -2.17805"/>
         </joint>
         <joint name="to_kinect_mesh" type="revolute">
@@ -287,5 +250,5 @@
             <child link="kinect_mesh"/>
             <limit lower="0" upper="0" effort="0" velocity="0"/>
-            <origin xyz="0 0 0.015" rpy="0 0 1.57"/>
+            <origin xyz="0.02 0 0" rpy="1.57 0 1.57"/>
         </joint>
         <link name ="kinect_frame"/>
